Commit message: added joint and control node

File: description/gazebo_control.xacro (robot description, xacro)
@@ -1,5 +1,5 @@
 <?xml version="1.0"?>
 <robot xmlns:xacro="http://www.ros.org/wiki/xacro"  name="robot">
-    <gazebo>
+  <gazebo>
     <plugin name="object_controller" filename="libgazebo_ros_planar_move.so">
       <commandTopic>cmd_vel</commandTopic>
@@ -10,3 +10,9 @@
     </plugin>
   </gazebo>
+  <gazebo reference="my_bot">
+  <plugin name="gazebo_ros_state" filename="libgazebo_ros_state.so">
+    <!-- Update rate, in Hz -->
+    <updateRate>10.0</updateRate>
+  </plugin>
+</gazebo>
 </robot>

File: description/lidar.xacro (robot description, xacro)
@@ -41,5 +41,5 @@
                 <range>
                     <min>0.3</min>
-                    <max>12</max>
+                    <max>5.0</max>
                 </range>
             </ray>

File: description/robot_core.xacro (robot description, xacro)
@@ -44,5 +44,5 @@
             <material name="white"/>
         </collision>
-        <visual>
+        <!-- <visual>
             <origin xyz="0.0 0.0 0.047" rpy="0.0 0.0 0.0"/>
             <geometry>
@@ -50,5 +50,5 @@
             </geometry>
             <material name="white"/>
-        </visual>
+        </visual> -->
     </link>
     <gazebo reference="chassis_link">
